File: sharp-lcd-27/sharp-lcd-27.kicad_sch (KiCad schematic)
At the start: 42 parts, among them J1 FH52-10S-0.5SH_99, J2 FH34SRJ-6S-0.5SH_50_, J3 USB_C_Programming, J4 Jack-DC, J6 Conn_01x06_Socket, Q2 BC817, Q3 BC817, SW1 RESET, SW2 BUTTON1, SW3 BUTTON2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

Commit message: #12 cleanup
Parts:
- added J5: Conn_01x04, footprint:QWIIC_JST_SH_BM04B-SRSS-TB_04x1.00mm, symbol Connector_Generic:Conn_01x04
- U3: footprint DRB8_2P4X1P65 -> footprint:TPS2113_2P4X1P65
Connections:
- net +3V3: now also J5.2 (Pin_2); no longer J1.6, J1.7
- net GND: now also J5.1 (Pin_1)
- net I2C_SCL: now also J5.4 (Pin_4)
- net I2C_SDA: now also J5.3 (Pin_3)
- net LCD_VCC_MUXOUT: now reaches C18.1, U3.7 (OUT), U5.3 (VI)
- net LCD_VCC_MUXOUT: now also J1.6, J1.7
- no-connect marks 10 -> 11
Other:
- note added: "QWIIC I2C Connector"
- note added: "UART Ext. Connector"
- note removed: "UART CONNECTION"
- moved on the sheet: H1, H2, H3, H4, J6

Commit message: #12 sharp 240x400 controller passes DRC
Parts:
- added R15: 10 K, Resistor_SMD:R_0603_1608Metric, symbol Device:R_Small
- added R3: 5.1k, Resistor_SMD:R_0402_1005Metric, symbol Device:R
- added SW4: BUTTON3, footprint:Alps_SKRK, symbol Switch:SW_Push
- added TP3: RTC_INT, TestPoint:TestPoint_Pad_1.0x1.0mm, symbol Connector:TestPoint
- J4: footprint Connector_JST:JST_ACH_BM02B-ACHSS-GAN-ETF_1x02-1MP_P1.20mm_Vertical -> Connector_JST:JST_EH_S2B-EH_1x02_P2.50mm_Horizontal
Connections:
- net +3V3: now also R15.1
- net GND: now also R3.2, SW4.2
- net at U7.1 (32KHZ): now also TP3.1
- net at J3.A5 (CC1): now also R3.1
- net BOOTMODE renamed IO_9
- net LCD_DISP: no longer names the net of J1.5, R14.1
- net LCD_DISP: no longer U1.16 (IO2)
- new net IO_2: R15.2, SW4.1, U1.16 (IO2)
- no-connect marks 11 -> 10
Other:
- note added: "BUTTON3"
- note added: "JP1 as default bridged Leave open IF Touch interrupt is used"
- note added: "LCD_DISP always on"
- note removed: "JP1 as default bridged Leave open IF Touch is used"
